File: ps2_MXODE.kicad_sch (KiCad schematic)
At the start: 79 parts, among them J1 USB_C_Receptacle_USB2.0_16P, J2 Conn_01x40, J3 Micro_SD_Card_Det_Hirose_DM3AT, J4 FPGA_JTAG, U1 STM32F405RGTx, U2 GW2AR-LV18QN88C8_I7, U3 W25Q64JVSS, U4 MT3520B, U5 MT3520B, Y1 Crystal, Y2 7050-27MHz

Commit message: Corrected schematic
Connections:
- net HACK: now also J2.38 (Pin_38), U2.41 (IOB43A); no longer J2.39 (Pin_39), U2.42 (IOB42B)
- net ~{CS_OUT}: now also J2.39 (Pin_39), U2.42 (IOB42B); no longer J2.38 (Pin_38), U2.41 (IOB43A)
Changed lines of the file:
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@@
 		)
 	)
-	(label "HACK"
-		(at 196.85 -67.31 0)
-		(effects
-			(font
-				(size 1.27 1.27)
-			)
-			(justify left bottom)
+	(label "~{CS_OUT}"
+		(at 347.98 3.81 180)
+		(effects
+			(font
+				(size 1.27 1.27)
+			)
+			(justify right bottom)
 		)
 	)
@@
 		)
 	)
-	(label "~{CS_OUT}"
-		(at 196.85 -69.85 0)
-		(effects
-			(font
-				(size 1.27 1.27)
-			)
-			(justify left bottom)
-		)
-	)
 	(label "TDI"
 		(at 408.94 -99.06 0)
@@
 		)
 	)
-	(label "HACK"
-		(at 347.98 3.81 180)
-		(effects
-			(font
-				(size 1.27 1.27)
-			)
-			(justify right bottom)
-		)
-	)
 	(label "A15"
 		(at 196.85 -151.13 0)
@@
 		)
 	)
+	(label "HACK"
+		(at 347.98 1.27 180)
+		(effects
+			(font
+				(size 1.27 1.27)
+			)
+			(justify right bottom)
+		)
+	)
 	(label "STM_MOSI"
 		(at 129.54 -109.22 0)
@@
 		)
 	)
+	(label "~{CS_OUT}"
+		(at 196.85 -67.31 0)
+		(effects
+			(font
+				(size 1.27 1.27)
+			)
+			(justify left bottom)
+		)
+	)
 	(label "VCCPLLR"
 		(at 408.94 -107.95 0)
@@
 		)
 	)
-	(label "~{CS_OUT}"
-		(at 347.98 1.27 180)
-		(effects
-			(font
-				(size 1.27 1.27)
-			)
-			(justify right bottom)
-		)
-	)
 	(label "TDO"
 		(at 454.66 -96.52 180)
@@
 		(effects
 			(font
+				(size 1.27 1.27)
+			)
+			(justify left bottom)
+		)
+	)
+	(label "HACK"
+		(at 196.85 -69.85 0)
+		(effects
+			(font
